File: LEOS-stack-template.kicad_sch (KiCad schematic)
At the start: 19 parts, among them J1 MicroFit_1x4, J2 MicroFit_1x4, U1 MCP2562FD, U2 MCP2518FD, Y1 40 MHz

Commit message: Set up EFM sheet with scattered op-amps
Other:
- added sheet EFM (EFM.kicad_sch)
Changed lines of the file:
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@@
+		)
+	)
+	(sheet
+		(at 118.11 130.81)
+		(size 111.76 31.75)
+		(exclude_from_sim no)
+		(in_bom yes)
+		(on_board yes)
+		(dnp no)
+		(fields_autoplaced yes)
+		(stroke
+			(width 0.1524)
+			(type solid)
+		)
+		(fill
+			(color 0 0 0 0.0000)
+		)
+		(property "Sheetname" "EFM"
+			(at 118.11 130.0984 0)
+			(effects
+				(font
+					(size 1.27 1.27)
+				)
+				(justify left bottom)
+			)
+		)
+		(property "Sheetfile" "EFM.kicad_sch"
+			(at 118.11 163.1446 0)
+			(effects
+				(font
+					(size 1.27 1.27)
+				)
+				(justify left top)
+			)
+		)
+		(instances
+			(project "LEOS-stack-template"
+				(path "/3703ddf2-8141-438d-86a8-1eaec9672d0d"
+					(page "2")
+				)
+			)
 		)
 	)
