File: LEOS-efm.kicad_pcb (KiCad board)
At the start: 2 copper layers, 100 x 100 mm, 22 parts, among them J1 MicroFit_1x4, J2 MicroFit_1x4, U1 MCP2562FD, U2 MCP2518FD, Y1 40 MHz

Commit message: v1.0
Parts:
- added C12: 220p, Capacitor_SMD:C_0805_2012Metric, F.Cu at (172.5, 122.5)
- added C13: 220p, Capacitor_SMD:C_0805_2012Metric, F.Cu at (177.4, 106.5)
- added C14: 220p, Capacitor_SMD:C_0805_2012Metric, F.Cu at (177.5, 122.5)
- added C15: 220p, Capacitor_SMD:C_0805_2012Metric, F.Cu at (172.4, 106.3)
- added C16: 0.1u, Capacitor_SMD:C_0603_1608Metric, F.Cu at (181.0, 96.7)
- added C17: 0.1u, Capacitor_SMD:C_0603_1608Metric, F.Cu at (180.5, 136.3)
- added J3: EFM 1, Connector_JST:JST_XH_S5B-XH-A_1x05_P2.50mm_Horizontal, F.Cu at (190.1, 138.0)
- added J4: EFM 2, Connector_JST:JST_XH_S5B-XH-A_1x05_P2.50mm_Horizontal, F.Cu at (190.1, 100.5)
- added R10: 1k, Resistor_SMD:R_0805_2012Metric, F.Cu at (180.4, 128.0)
- added R11: 1k, Resistor_SMD:R_0805_2012Metric, F.Cu at (173.1, 101.0)
- added R12: 20M, Resistor_SMD:R_0805_2012Metric, F.Cu at (172.5, 103.5)
- added R13: 1k, Resistor_SMD:R_0805_2012Metric, F.Cu at (169.6, 101.0)
- added R14: 10k, Resistor_SMD:R_0805_2012Metric, F.Cu at (154.1, 120.5)
- added R15: 10k, Resistor_SMD:R_0805_2012Metric, F.Cu at (157.6, 120.5)
- added R2: 1k, Resistor_SMD:R_0805_2012Metric, F.Cu at (173.3, 128.0)
- added R3: 20M, Resistor_SMD:R_0805_2012Metric, F.Cu at (172.6, 125.5)
- added R4: 1k, Resistor_SMD:R_0805_2012Metric, F.Cu at (169.9, 128.0)
- added R5: 1k, Resistor_SMD:R_0805_2012Metric, F.Cu at (176.6, 101.0)
- added R6: 20M, Resistor_SMD:R_0805_2012Metric, F.Cu at (177.4, 103.5)
- added R7: 1k, Resistor_SMD:R_0805_2012Metric, F.Cu at (180.0, 101.0)
- added R8: 1k, Resistor_SMD:R_0805_2012Metric, F.Cu at (176.8, 128.0)
- added R9: 20M, Resistor_SMD:R_0805_2012Metric, F.Cu at (177.5, 125.5)
- added U3: TL074, Package_DIP:DIP-14_W7.62mm, F.Cu at (167.4, 118.0)
- added U4: TL071, Package_DIP:DIP-8_W7.62mm, F.Cu at (151.0, 118.1)
- added U7: MCP3428 - EFM1, Package_SO:SOIC-14_3.9x8.7mm_P1.27mm, F.Cu at (175.0, 134.5)
- added U8: MCP3428 - EFM2, Package_SO:SOIC-14_3.9x8.7mm_P1.27mm, F.Cu at (175.5, 94.5)
Connections:
- A1 pad 11: unconnected-(A1-GPIO8-Pad11) -> /EFM/SDA
- A1 pad 12: unconnected-(A1-GPIO9-Pad12) -> /EFM/SCL
Routing:
- net +5V: track 107.8 -> 289.7 mm, vias 0 -> 1
- net /EFM/SDA: track 0.00 -> 120.4 mm, vias 0 -> 2
- net /EFM/SCL: track 0.00 -> 119.4 mm, vias 0 -> 4
- net +2.5V: track 0.00 -> 49.8 mm
- net /EFM/EFM1_PHASE1: track 0.00 -> 24.8 mm
- net /EFM/EFM2_PHASE2: track 0.00 -> 21.2 mm
- net /EFM/EFM1_IR: track 0.00 -> 19.8 mm
- net Net-(U8-CH1+): track 0.00 -> 19.6 mm, vias 0 -> 2
- net /EFM/EFM2_IR: track 0.00 -> 18.3 mm
- net Net-(U7-CH1-): track 0.00 -> 17.5 mm, vias 0 -> 2
- net /EFM/EFM2_PHASE1: track 0.00 -> 16.7 mm
- net /EFM/EFM1_PHASE2: track 0.00 -> 16.1 mm, vias 0 -> 2
- net Net-(U8-CH1-): track 0.00 -> 15.0 mm
- net Net-(U7-CH1+): track 0.00 -> 15.0 mm
- net Net-(C12-Pad2): track 0.00 -> 11.7 mm
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Other:
- board text added: "02/20/2026"
- board text added: "EFM 1"
- board text added: "EFM 2"
- board text added: "LEOS EFM Rev.1"
- board text removed: "LEOS CHANGE THIS NAME Rev. 3"
