File: LEOS-efm.kicad_pcb (KiCad board)
At the start: 2 copper layers, 100 x 100 mm, 48 parts, among them J1 MicroFit_1x4, J2 MicroFit_1x4, J3 EFM 1, J4 EFM 2, U1 MCP2562FD, U2 MCP2518FD, U3 TL074, U4 TL071, U7 MCP3428 - EFM1, U8 MCP3428 - EFM2, Y1 40 MHz

Commit message: New v3.0 template
Parts:
- removed C10, C16, C17: 0.1u, Capacitor_SMD:C_0603_1608Metric
- removed C11: 10u, Capacitor_SMD:C_0805_2012Metric
- removed C12, C13, C14, C15: 220p, Capacitor_SMD:C_0805_2012Metric
- removed the C4 at (139.5, 67.7)
- removed the C5 at (125.7, 76.0)
- removed the C6 at (125.7, 78.0)
- removed the C7 at (121.7, 68.5)
- removed J3: EFM 1, Connector_JST:JST_XH_S5B-XH-A_1x05_P2.50mm_Horizontal
- removed J4: EFM 2, Connector_JST:JST_XH_S5B-XH-A_1x05_P2.50mm_Horizontal
- removed R10, R11, R13, R2, R4, R5, R7, R8: 1k, Resistor_SMD:R_0805_2012Metric
- removed R12, R3, R6, R9: 20M, Resistor_SMD:R_0805_2012Metric
- removed R14, R15: 10k, Resistor_SMD:R_0805_2012Metric
- removed U3: TL074, Package_DIP:DIP-14_W7.62mm
- removed U4: TL071, Package_DIP:DIP-8_W7.62mm
- removed U7: MCP3428 - EFM1, Package_SO:SOIC-14_3.9x8.7mm_P1.27mm
- removed U8: MCP3428 - EFM2, Package_SO:SOIC-14_3.9x8.7mm_P1.27mm
- added C1: 0.1u, Capacitor_SMD:C_0805_2012Metric, F.Cu at (123.5, 68.5)
- added C2: 0.1u, Capacitor_SMD:C_0805_2012Metric, F.Cu at (137.5, 68.0)
- A1: footprint Module:RaspberryPi_Pico_Common_THT -> Module:RaspberryPi_Pico_Common_Unspecified
- C3: footprint Capacitor_SMD:C_0603_1608Metric -> Capacitor_SMD:C_0805_2012Metric
- C4: renamed from C2; footprint Capacitor_SMD:C_0603_1608Metric -> Capacitor_SMD:C_0805_2012Metric
- C5: renamed from C1; footprint Capacitor_SMD:C_0603_1608Metric -> Capacitor_SMD:C_0805_2012Metric
- C6: renamed from C8; footprint Capacitor_SMD:C_0805_2012Metric -> Capacitor_SMD:C_1206_3216Metric
- C7: renamed from C9; footprint Capacitor_SMD:C_0805_2012Metric -> Capacitor_SMD:C_1206_3216Metric
- moved A1 25.6 mm to (173.6, 67.1)
- moved C3 16.4 mm to (123.5, 76.2), turned to 0 degrees
- moved R1 1.00 mm to (118.0, 68.2)
- moved TP1 1.00 mm to (118.0, 79.0)
- moved TP2 1.00 mm to (118.0, 65.0)
- moved TP3 1.00 mm to (118.0, 85.0)
- moved TP4 1.00 mm to (118.0, 59.0)
- moved C7 0.73 mm to (113.8, 73.0)
- moved C6 0.53 mm to (113.8, 70.5)
- moved C4 0.06 mm to (135.0, 77.2)
- renumbered U2 to U1, U1 to U2
Connections:
- net Net-(U1-RXD) renamed /CANbus/RXCAN
- net Net-(U1-TXD) renamed /CANbus/TXCAN
- A1 pad 11: /EFM/SDA -> unconnected-(A1-GPIO8-Pad11)
- A1 pad 12: /EFM/SCL -> unconnected-(A1-GPIO9-Pad12)
- C3 pad 1: VDD -> +5V
Routing:
- net +5V: track 289.7 -> 104.0 mm, vias 1 -> 0
- net /EFM/SDA: track 120.4 -> 0.00 mm, vias 2 -> 0
- net /EFM/SCL: track 119.4 -> 0.00 mm, vias 4 -> 0
- net +2.5V: track 49.8 -> 0.00 mm
- net /EFM/EFM1_PHASE1: track 24.8 -> 0.00 mm
- net /EFM/EFM2_PHASE2: track 21.2 -> 0.00 mm
- net /EFM/EFM1_IR: track 19.8 -> 0.00 mm
- net Net-(U8-CH1+): track 19.6 -> 0.00 mm, vias 2 -> 0
- net /EFM/EFM2_IR: track 18.3 -> 0.00 mm
- net Net-(U7-CH1-): track 17.5 -> 0.00 mm, vias 2 -> 0
- net /EFM/EFM2_PHASE1: track 16.7 -> 0.00 mm
- net /EFM/EFM1_PHASE2: track 16.1 -> 0.00 mm, vias 2 -> 0
- net Net-(U8-CH1-): track 15.0 -> 0.00 mm
- net Net-(U7-CH1+): track 15.0 -> 0.00 mm
- net /CANbus/CAN-: track 51.3 -> 39.1 mm
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Other:
- board text added: "${ISSUE_DATE}"
- board text added: "Be sure to update the information block at the bottom of the page! (Then delete me)"
- board text added: "LEOS ${TITLE} Rev ${REVISION}"
- board text added: "Populate R1 with 120Ω if board is at end of bus."
- board text removed: "02/20/2026"
- board text removed: "EFM 1"
- board text removed: "EFM 2"
- board text removed: "LEOS EFM Rev.1"

Commit message: Add two hall effect sensor circuit and two EFM opamp to differential ADC circuit
Parts:
- added J3: Hall1_IN, Connector_JST:JST_XH_S3B-XH-A-1_1x03_P2.50mm_Horizontal, F.Cu at (206.5, 123.7)
- added J4: Hall2_IN, Connector_JST:JST_XH_S3B-XH-A-1_1x03_P2.50mm_Horizontal, F.Cu at (218.4, 123.7)
- added J5: Conn_01x03_Pin, Connector_JST:JST_XH_S3B-XH-A-1_1x03_P2.50mm_Horizontal, F.Cu at (206.5, 94.9)
- added J6: Conn_01x03_Pin, Connector_JST:JST_XH_S3B-XH-A-1_1x03_P2.50mm_Horizontal, F.Cu at (218.4, 94.9)
- added J7: Conn_01x03_Pin, Connector_JST:JST_XH_S3B-XH-A-1_1x03_P2.50mm_Horizontal, F.Cu at (230.4, 94.9)
- added J8: Conn_01x03_Pin, Connector_JST:JST_XH_S3B-XH-A-1_1x03_P2.50mm_Horizontal, F.Cu at (242.3, 94.9)
- added R10: 100k, Resistor_SMD:R_1206_3216Metric_Pad1.30x1.75mm_HandSolder, F.Cu at (217.9, 105.2)
- added R11: 100k, Resistor_SMD:R_1206_3216Metric_Pad1.30x1.75mm_HandSolder, F.Cu at (217.9, 108.5)
- added R12: 50, Resistor_SMD:R_1206_3216Metric_Pad1.30x1.75mm_HandSolder, F.Cu at (217.9, 111.8)
- added R13: 50, Resistor_SMD:R_1206_3216Metric_Pad1.30x1.75mm_HandSolder, F.Cu at (217.9, 115.1)
- added R2: 1k, Resistor_SMD:R_1206_3216Metric_Pad1.30x1.75mm_HandSolder, F.Cu at (206.0, 105.2)
- added R3: 100k, Resistor_SMD:R_1206_3216Metric_Pad1.30x1.75mm_HandSolder, F.Cu at (206.0, 108.5)
- added R4: 50, Resistor_SMD:R_1206_3216Metric_Pad1.30x1.75mm_HandSolder, F.Cu at (206.0, 111.8)
- added R5: 1k, Resistor_SMD:R_1206_3216Metric_Pad1.30x1.75mm_HandSolder, F.Cu at (206.0, 115.1)
- added R6: 100k, Resistor_SMD:R_1206_3216Metric_Pad1.30x1.75mm_HandSolder, F.Cu at (211.9, 105.2)
- added R7: 50, Resistor_SMD:R_1206_3216Metric_Pad1.30x1.75mm_HandSolder, F.Cu at (211.9, 108.5)
- added R8: 1k, Resistor_SMD:R_1206_3216Metric_Pad1.30x1.75mm_HandSolder, F.Cu at (211.9, 111.8)
- added R9: 1k, Resistor_SMD:R_1206_3216Metric_Pad1.30x1.75mm_HandSolder, F.Cu at (211.9, 115.1)
- added U3: OPA2333xxD, Package_SO:SOIC-8_3.9x4.9mm_P1.27mm, F.Cu at (225.1, 106.9)
- added U4: ADS1220xPW, Package_SO:TSSOP-16_4.4x5mm_P0.65mm, F.Cu at (234.1, 106.8)
- added U5: OPA2333xxD, Package_SO:SOIC-8_3.9x4.9mm_P1.27mm, F.Cu at (225.1, 113.5)
Connections:
- A1 pad 14: unconnected-(A1-GPIO10-Pad14) -> /GAIN100stage/SCLK
- A1 pad 15: unconnected-(A1-GPIO11-Pad15)_1 -> /GAIN100stage/DIN
- A1 pad 16: unconnected-(A1-GPIO12-Pad16) -> /GAIN100stage/DOUT
- A1 pad 17: unconnected-(A1-GPIO13-Pad17) -> /GAIN100stage/CS
- A1 pad 21: unconnected-(A1-GPIO16-Pad21)_1 -> /HALL1_IN
- A1 pad 22: unconnected-(A1-GPIO17-Pad22)_1 -> /HALL2_IN

Commit message: Finish layout and routing. Fix backward opamp terminals
Parts:
- removed J3: Hall1_IN, Connector_JST:JST_XH_S3B-XH-A-1_1x03_P2.50mm_Horizontal
- removed J4: Hall2_IN, Connector_JST:JST_XH_S3B-XH-A-1_1x03_P2.50mm_Horizontal
- removed J5, J6, J7, J8: Conn_01x03_Pin, Connector_JST:JST_XH_S3B-XH-A-1_1x03_P2.50mm_Horizontal
- added C10: 0.1u, Capacitor_SMD:C_0805_2012Metric, F.Cu at (182.0, 123.0)
- added C12: 0.1u, Capacitor_SMD:C_0805_2012Metric, F.Cu at (162.2, 106.2)
- added C13: 4.7u, Capacitor_SMD:C_1206_3216Metric, F.Cu at (166.0, 106.2)
- added C14: 4.7u, Capacitor_SMD:C_1206_3216Metric, F.Cu at (162.0, 81.5)
- added C15: 4.7u, Capacitor_SMD:C_1206_3216Metric, F.Cu at (172.5, 81.5)
- added C8: 0.1u, Capacitor_SMD:C_0805_2012Metric, F.Cu at (182.0, 89.8)
- added C9: 4.7u, Capacitor_SMD:C_1206_3216Metric, F.Cu at (174.5, 105.0)
- added J10: S3B-XH-A-1, Connector_JST:JST_XH_S3B-XH-A-1_1x03_P2.50mm_Horizontal, F.Cu at (191.0, 97.8)
- added J11: S3B-XH-A-1, Connector_JST:JST_XH_S3B-XH-A-1_1x03_P2.50mm_Horizontal, F.Cu at (191.0, 108.8)
- added J12: B3B-XH-A, Connector_JST:JST_XH_B3B-XH-A_1x03_P2.50mm_Vertical, F.Cu at (155.5, 140.5)
- added J13: B3B-XH-A, Connector_JST:JST_XH_B3B-XH-A_1x03_P2.50mm_Vertical, F.Cu at (166.5, 140.5)
- added J14: S3B-XH-A-1, Connector_JST:JST_XH_S3B-XH-A-1_1x03_P2.50mm_Horizontal, F.Cu at (191.0, 141.8)
- added J15: S3B-XH-A-1, Connector_JST:JST_XH_S3B-XH-A-1_1x03_P2.50mm_Horizontal, F.Cu at (191.0, 130.8)
- added J16: S3B-XH-A-1, Connector_JST:JST_XH_S3B-XH-A-1_1x03_P2.50mm_Horizontal, F.Cu at (191.0, 119.8)
- added J9: S3B-XH-A-1, Connector_JST:JST_XH_S3B-XH-A-1_1x03_P2.50mm_Horizontal, F.Cu at (191.0, 86.8)
- added R14: 100k, Resistor_SMD:R_1206_3216Metric, F.Cu at (172.5, 119.0)
- added R15: 100k, Resistor_SMD:R_1206_3216Metric, F.Cu at (172.5, 126.8)
- added R16: 33, Resistor_SMD:R_1206_3216Metric, F.Cu at (172.5, 121.5)
- added R17: 33, Resistor_SMD:R_1206_3216Metric, F.Cu at (172.5, 124.2)
- added R20: 10k, Resistor_SMD:R_1206_3216Metric, F.Cu at (164.7, 81.5)
- added R21: 10k, Resistor_SMD:R_1206_3216Metric, F.Cu at (169.8, 81.5)
- R10, R11: value 100k -> 1k; footprint Resistor_SMD:R_1206_3216Metric_Pad1.30x1.75mm_HandSolder -> Resistor_SMD:R_1206_3216Metric
- R12, R13, R4: value 50 -> 1k; footprint Resistor_SMD:R_1206_3216Metric_Pad1.30x1.75mm_HandSolder -> Resistor_SMD:R_1206_3216Metric
- R2: value 1k -> 10k; footprint Resistor_SMD:R_1206_3216Metric_Pad1.30x1.75mm_HandSolder -> Resistor_SMD:R_1206_3216Metric
- R3: value 100k -> 10k; footprint Resistor_SMD:R_1206_3216Metric_Pad1.30x1.75mm_HandSolder -> Resistor_SMD:R_1206_3216Metric
- R5, R6: footprint Resistor_SMD:R_1206_3216Metric_Pad1.30x1.75mm_HandSolder -> Resistor_SMD:R_1206_3216Metric
- R7: value 50 -> 100k; footprint Resistor_SMD:R_1206_3216Metric_Pad1.30x1.75mm_HandSolder -> Resistor_SMD:R_1206_3216Metric
- R8, R9: value 1k -> 33; footprint Resistor_SMD:R_1206_3216Metric_Pad1.30x1.75mm_HandSolder -> Resistor_SMD:R_1206_3216Metric
- U3, U5: value OPA2333xxD -> OPA2333AID
- U4: value ADS1220xPW -> ADS1220IPW
- moved U4 75.8 mm to (158.2, 106.2), turned to 90 degrees
- moved U3 50.1 mm to (178.0, 89.8), turned to -90 degrees
- moved U5 48.0 mm to (178.0, 123.0), turned to -90 degrees
- moved R9 46.2 mm to (172.5, 91.0), turned to 180 degrees
- moved R8 45.9 mm to (172.5, 88.2), turned to 180 degrees
- moved R6 44.0 mm to (172.5, 85.8), turned to 180 degrees
- moved R7 42.2 mm to (172.5, 93.5), turned to 180 degrees
- moved R13 41.9 mm to (178.0, 128.0), turned to 180 degrees
- moved R11 41.0 mm to (177.0, 105.0), turned to -90 degrees
- moved R12 40.2 mm to (178.0, 117.2), turned to 180 degrees
- moved R4 39.5 mm to (178.0, 84.0), turned to 180 degrees
- moved R10 38.4 mm to (179.5, 105.0), turned to 90 degrees
- moved R3 34.6 mm to (182.2, 133.8), turned to 180 degrees
- moved R5 34.5 mm to (178.0, 95.0), turned to 180 degrees
- moved R2 24.2 mm to (182.2, 100.5), turned to 180 degrees
Connections:
- net /GAIN100stage/CS renamed /ADC/CS
- net /GAIN100stage/DIN renamed /ADC/MOSI
- net /GAIN100stage/DOUT renamed /ADC/MISO
- net /GAIN100stage/SCLK renamed /ADC/SCLK
- A1 pad 21: /HALL1_IN -> /EFM0_HALL
- A1 pad 22: /HALL2_IN -> /EFM1_HALL
- A1 pad 25: unconnected-(A1-GPIO19-Pad25) -> /ADC/~{DRDY}
- A1 pad 27: unconnected-(A1-GPIO21-Pad27)_1 -> Net-(A1-GPIO21)
- A1 pad 29: unconnected-(A1-GPIO22-Pad29) -> Net-(A1-GPIO22)
- R10 pad 1: Net-(U5A-+) -> VDD
- R10 pad 2: Net-(R10-Pad2) -> /ADC/V_{mid}
- R11 pad 1: Net-(U5B-+) -> /ADC/V_{mid}
- R11 pad 2: Net-(R11-Pad2) -> GND
- R12 pad 1: Net-(R10-Pad2) -> /EFM1_SENSE
- R12 pad 2: Net-(U4-AIN2) -> Net-(U5A--)
- R13 pad 1: Net-(R11-Pad2) -> /EFM1_REF
- R13 pad 2: Net-(U4-AIN3/REFN1) -> Net-(U5B--)
- R2 pad 1: Net-(J5-Pin_2) -> VDD
- R2 pad 2: Net-(U3A-+) -> /EFM0_HALL
- R3 pad 1: Net-(U3A-+) -> VDD
- R3 pad 2: Net-(R3-Pad2) -> /EFM1_HALL
- R4 pad 1: Net-(R3-Pad2) -> /EFM0_SENSE
- R4 pad 2: Net-(U4-AIN0/REFP1) -> Net-(U3A--)
- R5 pad 1: Net-(J6-Pin_2) -> /EFM0_REF
- R5 pad 2: Net-(U3B-+) -> Net-(U3B--)
- R6 pad 1: Net-(U3B-+) -> Net-(U3A--)
- R7 pad 1: Net-(R6-Pad2) -> Net-(U3B--)
- R7 pad 2: Net-(U4-AIN1) -> Net-(R7-Pad2)
- R8 pad 1: Net-(J7-Pin_2) -> Net-(R6-Pad2)
- R8 pad 2: Net-(U5A-+) -> /ADC/SENSE0
- R9 pad 1: Net-(J8-Pin_2) -> Net-(R7-Pad2)
- R9 pad 2: Net-(U5B-+) -> /ADC/REF0
- U3 pad 1: Net-(R3-Pad2) -> Net-(R6-Pad2)
- U3 pad 2: GND -> Net-(U3A--)
- U3 pad 3: Net-(U3A-+) -> /ADC/V_{mid}
- U3 pad 5: Net-(U3B-+) -> /ADC/V_{mid}
- U3 pad 6: GND -> Net-(U3B--)
- U3 pad 7: Net-(R6-Pad2) -> Net-(R7-Pad2)
- U4 pad 10: Net-(U4-AIN1) -> /ADC/REF0
- U4 pad 11: Net-(U4-AIN0/REFP1) -> /ADC/SENSE0
- U4 pad 14: unconnected-(U4-~{DRDY}-Pad14) -> /ADC/~{DRDY}
- U4 pad 6: Net-(U4-AIN3/REFN1) -> /ADC/REF1
- U4 pad 7: Net-(U4-AIN2) -> /ADC/SENSE1
- U5 pad 1: Net-(R10-Pad2) -> Net-(R14-Pad2)
- U5 pad 2: GND -> Net-(U5A--)
- U5 pad 3: Net-(U5A-+) -> /ADC/V_{mid}
- U5 pad 5: Net-(U5B-+) -> /ADC/V_{mid}
- U5 pad 6: GND -> Net-(U5B--)
- U5 pad 7: Net-(R11-Pad2) -> Net-(R15-Pad2)
Routing:
- net VDD: track 90.8 -> 313.1 mm
- net /EFM1_HALL: track 0.00 -> 91.4 mm
- net /EFM0_CAL: track 0.00 -> 73.6 mm, vias 0 -> 7
- net /EFM1_CAL: track 0.00 -> 70.6 mm, vias 0 -> 7
- net /EFM0_HALL: track 0.00 -> 66.9 mm, vias 0 -> 2
- net /ADC/SCLK: track 0.00 -> 60.2 mm, vias 0 -> 1
- net /ADC/V_{mid}: track 0.00 -> 57.7 mm, vias 0 -> 10
- net /ADC/CS: track 0.00 -> 52.3 mm, vias 0 -> 1
- net /ADC/MOSI: track 0.00 -> 49.7 mm, vias 0 -> 1
- net /ADC/MISO: track 0.00 -> 46.4 mm, vias 0 -> 1
- net /ADC/~{DRDY}: track 0.00 -> 27.6 mm
- net /ADC/SENSE0: track 0.00 -> 20.0 mm
- net /ADC/REF1: track 0.00 -> 20.0 mm
- net /ADC/REF0: track 0.00 -> 18.1 mm
- net /ADC/SENSE1: track 0.00 -> 17.9 mm
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Other:
- board text added: "C8"
- board text added: "EFM0 CALIBRATION"
- board text added: "EFM0 HALL EFFECT"
- board text added: "EFM0 REFERENCE"
- board text added: "EFM0 SENSING"
- board text added: "EFM1 CALIBRATION"
- board text added: "EFM1 HALL EFFECT"
- board text added: "EFM1 REFERENCE"
- board text added: "EFM1 SENSING"
- board text removed: "Be sure to update the information block at the bottom of the page! (Then delete me)"

Commit message: Final Production Schematic/PCB Fall 2026
Parts:
- added C11: 3.3u, Capacitor_SMD:C_1206_3216Metric, F.Cu at (182.8, 84.0)
- added C16: 3.3u, Capacitor_SMD:C_1206_3216Metric, F.Cu at (182.7, 117.2)
- added C17: 3.3u, Capacitor_SMD:C_1206_3216Metric, F.Cu at (182.7, 95.0)
- added C18: 3.3u, Capacitor_SMD:C_1206_3216Metric, F.Cu at (182.8, 128.0)
- R12, R13, R4, R5: value 1k -> 10k
- R14, R15, R6, R7: value 100k -> 1M
Connections:
- R12 pad 1: /EFM1_SENSE -> Net-(C16-Pad2)
- R13 pad 1: /EFM1_REF -> Net-(C18-Pad2)
- R4 pad 1: /EFM0_SENSE -> Net-(C11-Pad2)
- R5 pad 1: /EFM0_REF -> Net-(C17-Pad2)
Routing:
- net /EFM0_SENSE: track 11.6 -> 6.38 mm
- net /EFM1_REF: track 11.6 -> 6.88 mm
- net /EFM1_SENSE: track 11.5 -> 6.80 mm
- net /EFM0_REF: track 11.6 -> 6.90 mm
- net Net-(C18-Pad2): track 0.00 -> 1.81 mm
- net Net-(C11-Pad2): track 0.00 -> 1.81 mm
- net Net-(C17-Pad2): track 0.00 -> 1.79 mm
- net Net-(C16-Pad2): track 0.00 -> 1.79 mm
Other:
- board text added: "EFM0 HALL"
- board text added: "EFM0 REF"
- board text added: "EFM1 HALL"
- board text added: "EFM1 REF"
- board text removed: "EFM0 HALL EFFECT"
- board text removed: "EFM0 REFERENCE"
- board text removed: "EFM1 HALL EFFECT"
- board text removed: "EFM1 REFERENCE"
