File: LEOS-efm.kicad_sch (KiCad schematic)
At the start: 3 parts

Commit message: v1.0
Connections:
- net EFM/SDA: now reaches A1.11 (GPIO8)
- net EFM/SCL: now reaches A1.12 (GPIO9)
- no-connect marks 26 -> 24
Other:
- added sheet EFM (efm.kicad_sch)
Changed lines of the file:
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@@
-	)
-	(no_connect
-		(at 124.46 109.22)
 	)
 	(no_connect
@@
 	)
 	(no_connect
-		(at 124.46 111.76)
-	)
-	(no_connect
 		(at 170.18 116.84)
 	)
@@
 	(wire
 		(pts
+			(xy 106.68 111.76) (xy 124.46 111.76)
+		)
+		(stroke
+			(width 0)
+			(type default)
+		)
+	)
+	(wire
+		(pts
+			(xy 104.14 114.3) (xy 104.14 109.22)
+		)
+		(stroke
+			(width 0)
+			(type default)
+		)
+	)
+	(wire
+		(pts
+			(xy 95.25 114.3) (xy 104.14 114.3)
+		)
+		(stroke
+			(width 0)
+			(type default)
+		)
+	)
+	(wire
+		(pts
 			(xy 142.24 57.15) (xy 142.24 66.04)
 		)
@@
 	(wire
 		(pts
+			(xy 106.68 116.84) (xy 106.68 111.76)
+		)
+		(stroke
+			(width 0)
+			(type default)
+		)
+	)
+	(wire
+		(pts
 			(xy 73.66 100.33) (xy 80.01 100.33)
 		)
@@
 		(pts
 			(xy 152.4 57.15) (xy 161.29 57.15)
+		)
+		(stroke
+			(width 0)
+			(type default)
+		)
+	)
+	(wire
+		(pts
+			(xy 104.14 109.22) (xy 124.46 109.22)
+		)
+		(stroke
+			(width 0)
+			(type default)
+		)
+	)
+	(wire
+		(pts
+			(xy 95.25 116.84) (xy 106.68 116.84)
 		)
 		(stroke
@@
 		)
 		(instances
-			(project "LEOS-stack-template"
+			(project "LEOS-efm"
 				(path "/3703ddf2-8141-438d-86a8-1eaec9672d0d"
 					(page "3")
@@
 		)
 		(instances
-			(project "LEOS-stack-template"
+			(project "LEOS-efm"
 				(path "/3703ddf2-8141-438d-86a8-1eaec9672d0d"
 					(page "2")
 				)
 			)
+		)
+	)
+	(sheet
+		(at 80.01 111.76)
+		(size 15.24 13.97)
+		(exclude_from_sim no)
+		(in_bom yes)
+		(on_board yes)
+		(dnp no)
+		(fields_autoplaced yes)
+		(stroke
+			(width 0.1524)
+			(type solid)
+		)
+		(fill
+			(color 0 0 0 0.0000)
+		)
+		(property "Sheetname" "EFM"
+			(at 80.01 111.0484 0)
+			(effects
+				(font
+					(size 1.27 1.27)
+				)
+				(justify left bottom)
+			)
+		)
+		(property "Sheetfile" "efm.kicad_sch"
+			(at 80.01 126.3146 0)
+			(effects
+				(font
+					(size 1.27 1.27)
+				)
+				(justify left top)
+			)
+		)
+		(pin "SCL" bidirectional
+			(at 95.25 116.84 0)
+			(effects
+				(font
+					(size 1.27 1.27)
+				)
+				(justify right)
+			)
+		)
+		(pin "SDA" bidirectional
+			(at 95.25 114.3 0)
+			(effects
+				(font
+					(size 1.27 1.27)
+				)
+				(justify right)
+			)
+		)
+		(instances
+			(project "LEOS-efm"
+				(path "/3703ddf2-8141-438d-86a8-1eaec9672d0d"
+					(page "4")
+				)
+			)
