File: LEOS-efm.kicad_sch (KiCad schematic)
At the start: 3 parts

Commit message: New v3.0 template
Parts:
- removed C10: 0.1u, Capacitor_SMD:C_0603_1608Metric, symbol Device:C
- removed C11: 10u, Capacitor_SMD:C_0805_2012Metric, symbol Device:C
- A1: footprint Module:RaspberryPi_Pico_Common_THT -> Module:RaspberryPi_Pico_Common_Unspecified
Connections:
- net EFM/SCL: no longer names the net of A1.12 (GPIO9)
- net EFM/SDA: no longer names the net of A1.11 (GPIO8)
- no-connect marks 24 -> 26
Other:
- removed sheet EFM
- note added: "Have Fun! Delete this box once you start designing."
- note added: "This is the schematic for a circuit board module used in the LEOS Stack. Other than the standard CAN networking chips and Raspberry Pi Pico, this is your blank slate for creating any application designs."
- note added: "When authoring new schematics, remember these key points: 1. Ensure your page information is up to date. - keep the revision number, page title, and supporting text up to date with the design. This document should be self-explanatory as often as possible. - Delete the help text in the root sheet. 2. Commit your work into GitHub - Make incremental changes to the schematic and layout, but ensure th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"

Commit message: Add two hall effect sensor circuit and two EFM opamp to differential ADC circuit
Parts:
- added J3: Hall1_IN, Connector_JST:JST_XH_S3B-XH-A-1_1x03_P2.50mm_Horizontal, symbol Connector:Conn_01x03_Pin
- added J4: Hall2_IN, Connector_JST:JST_XH_S3B-XH-A-1_1x03_P2.50mm_Horizontal, symbol Connector:Conn_01x03_Pin
Connections:
- net GND: now also J3.3 (Pin_3), J4.3 (Pin_3)
- net VDD: now also J3.1 (Pin_1), J4.1 (Pin_1)
- net GAIN100stage/SCLK: now reaches A1.14 (GPIO10)
- net GAIN100stage/DIN: now reaches A1.15 (GPIO11)
- net GAIN100stage/DOUT: now reaches A1.16 (GPIO12)
- net GAIN100stage/CS: now reaches A1.17 (GPIO13)
- net HALL1_IN: now reaches A1.21 (GPIO16)
- net HALL1_IN: now also J3.2 (Pin_2)
- net HALL2_IN: now reaches A1.22 (GPIO17)
- net HALL2_IN: now also J4.2 (Pin_2)
- no-connect marks 26 -> 20
Other:
- added sheet GAIN100stage (GAIN100stage.kicad_sch)

Commit message: Finish layout and routing. Fix backward opamp terminals
Parts:
- removed J3: Hall1_IN, Connector_JST:JST_XH_S3B-XH-A-1_1x03_P2.50mm_Horizontal, symbol Connector:Conn_01x03_Pin
- removed J4: Hall2_IN, Connector_JST:JST_XH_S3B-XH-A-1_1x03_P2.50mm_Horizontal, symbol Connector:Conn_01x03_Pin
- added C14, C15: 4.7u, Capacitor_SMD:C_1206_3216Metric, symbol Device:C
- added J10, J11, J14, J15, J16, J9: S3B-XH-A-1, Connector_JST:JST_XH_S3B-XH-A-1_1x03_P2.50mm_Horizontal, symbol Connector_Generic:Conn_01x03
- added J12, J13: B3B-XH-A, Connector_JST:JST_XH_B3B-XH-A_1x03_P2.50mm_Vertical, symbol Connector_Generic:Conn_01x03
- added R2, R20, R21, R3: 10k, Resistor_SMD:R_1206_3216Metric, symbol Device:R_US
Connections:
- net GND: now also C14.2, C15.2, J10.3 (Pin_3), J11.3 (Pin_3), J12.3 (Pin_3), J13.3 (Pin_3), J14.3 (Pin_3), J15.3 (Pin_3), J16.3 (Pin_3), J9.3 (Pin_3)
- net VDD: now also J10.1 (Pin_1), J11.1 (Pin_1), J12.1 (Pin_1), J13.1 (Pin_1), J14.1 (Pin_1), J15.1 (Pin_1), J16.1 (Pin_1), J9.1 (Pin_1), R2.1, R3.1
- net ADC/~{DRDY}: now reaches A1.25 (GPIO19)
- net at A1.27 (GPIO21): now also R20.1
- net at A1.29 (GPIO22): now also R21.1
- net ADC/DIN renamed ADC/MOSI
- net ADC/DOUT renamed ADC/MISO
- net HALL1_IN renamed EFM0_HALL
- net EFM0_HALL: now also J11.2 (Pin_2), R2.2
- net HALL2_IN renamed EFM1_HALL
- net EFM1_HALL: now also J14.2 (Pin_2), R3.2
- new net EFM0_CAL: C14.1, J12.2 (Pin_2), R20.2
- new net EFM0_REF: J10.2 (Pin_2)
- new net EFM0_SENSE: J9.2 (Pin_2)
- new net EFM1_CAL: C15.1, J13.2 (Pin_2), R21.2
- new net EFM1_REF: J15.2 (Pin_2)
- new net EFM1_SENSE: J16.2 (Pin_2)
- no-connect marks 20 -> 17
Other:
- sheet GAIN100stage renamed ADC
- added sheet Electrode Amplifier 0 (opamp.kicad_sch)
- added sheet Electrode Amplifier 1 (opamp.kicad_sch)
- sheet ADC: file GAIN100stage.kicad_sch -> adc.kicad_sch
- sheet ADC ports: added MISO, MOSI, REF0, REF1, SENSE0, SENSE1, V_{mid}, ~{DRDY}; removed DIN, DOUT
- note added: "Digital hall effect sensors are open-collector outputs."
- note added: "PWM RC Lowpass f_{c} = 3.39Hz"
- note added: "Used as programmable voltage (0-3.3V) for EFM Calibration Plate"
- note removed: "Have Fun! Delete this box once you start designing."
- note removed: "This is the schematic for a circuit board module used in the LEOS Stack. Other than the standard CAN networking chips and Raspberry Pi Pico, this is your blank slate for creating any application designs."
- note removed: "When authoring new schematics, remember these key points: 1. Ensure your page information is up to date. - keep the revision number, page title, and supporting text up to date with the design. This document should be self-explanatory as often as possible. - Delete the help text in the root sheet. 2. Commit your work into GitHub - Make incremental changes to the schematic and layout, but ensure th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"
- title: LEOS Microcontroller -> LEOS EFM
