File: connectors.kicad_sch (KiCad schematic)
At the start: 7 parts, among them J1 MicroFit_1x4, J2 MicroFit_1x4

Commit message: New v3.0 template
Parts:
- C6: renamed from C8; footprint Capacitor_SMD:C_0805_2012Metric -> Capacitor_SMD:C_1206_3216Metric; Digikey 1276-CL21A226MAYNNNECT-ND -> 1276-3148-1-ND; LCSC C29936 -> C6142744; MPN CL21A226MAYNNNE -> CL31B226MPHNNNE
- C7: renamed from C9; footprint Capacitor_SMD:C_0805_2012Metric -> Capacitor_SMD:C_1206_3216Metric; Digikey 1276-CL21A226MAYNNNECT-ND -> 1276-3148-1-ND; LCSC C29936 -> C6142744; MPN CL21A226MAYNNNE -> CL31B226MPHNNNE
- R1, TP3, TP4: now left out of the parts list
