File: opamp.kicad_sch (KiCad schematic)
At the start: 8 parts, among them U3 OPA2333AID

Commit message: Final Production Schematic/PCB Fall 2026
Parts:
- added C11, C17: 3.3u, Capacitor_SMD:C_1206_3216Metric, symbol Device:C
- R4, R5: value 1k -> 10k
- R6, R7: value 100k -> 1M
Connections:
- net REF: now also C17.1; no longer R5.1
- net SENSE: now also C11.1; no longer R4.1
- new net: C17.2, R5.1
- new net: C11.2, R4.1
Changed lines of the file:
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@@
+	(wire
+		(pts
+			(xy 67.31 81.28) (xy 69.85 81.28)
+		)
+		(stroke
+			(width 0)
+			(type default)
+		)
+	)
 	(wire
 		(pts
@@
 	(wire
 		(pts
-			(xy 62.23 81.28) (xy 69.85 81.28)
+			(xy 52.07 81.28) (xy 59.69 81.28)
 		)
 		(stroke
@@
 	(wire
 		(pts
-			(xy 62.23 48.26) (xy 69.85 48.26)
+			(xy 52.07 48.26) (xy 59.69 48.26)
 		)
 		(stroke
@@
 		(pts
 			(xy 105.41 50.8) (xy 107.95 50.8)
+		)
+		(stroke
+			(width 0)
+			(type default)
+		)
+	)
+	(wire
+		(pts
+			(xy 67.31 48.26) (xy 69.85 48.26)
 		)
 		(stroke
@@
 	(hierarchical_label "SENSE"
 		(shape input)
-		(at 62.23 48.26 180)
+		(at 52.07 48.26 180)
 		(effects
 			(font
@@
 	(hierarchical_label "REF"
 		(shape input)
-		(at 62.23 81.28 180)
+		(at 52.07 81.28 180)
 		(effects
 			(font
@@
 			)
 			(justify right)
+		)
+	)
+	(symbol
+		(lib_id "Device:C")
+		(at 63.5 81.28 90)
+		(unit 1)
+		(body_style 1)
+		(exclude_from_sim no)
+		(in_bom yes)
+		(on_board yes)
+		(in_pos_files yes)
+		(dnp no)
+		(fields_autoplaced yes)
+		(property "Reference" "C17"
+			(at 63.5 73.66 90)
+			(show_name no)
+			(do_not_autoplace no)
+			(effects
+				(font
+					(size 1.27 1.27)
+				)
+			)
+		)
+		(property "Value" "3.3u"
+			(at 63.5 76.2 90)
+			(show_name no)
+			(do_not_autoplace no)
+			(effects
+				(font
+					(size 1.27 1.27)
+				)
+			)
+		)
+		(property "Footprint" "Capacitor_SMD:C_1206_3216Metric"
+			(at 67.31 80.3148 0)
+			(hide yes)
+			(show_name no)
+			(do_not_autoplace no)
+			(effects
+				(font
+					(size 1.27 1.27)
+				)
+			)
+		)
+		(property "Datasheet" ""
+			(at 63.5 81.28 0)
+			(hide yes)
+			(show_name no)
+			(do_not_autoplace no)
+			(effects
+				(font
+					(size 1.27 1.27)
+				)
+			)
+		)
+		(property "Description" "Unpolarized capacitor"
+			(at 63.5 81.28 0)
+			(hide yes)
+			(show_name no)
+			(do_not_autoplace no)
+			(effects
+				(font
+					(size 1.27 1.27)
+				)
+			)
+		)
+		(pin "1"
+		)
+		(pin "2"
+		)
+		(instances
+			(project "LEOS-efm"
+				(path "/3703ddf2-8141-438d-86a8-1eaec9672d0d/63365fd5-9ed8-4ace-be7f-754e14efcbff"
+					(reference "C17")
+					(unit 1)
+				)
+				(path "/3703ddf2-8141-438d-86a8-1eaec9672d0d/fd5efc03-4429-4730-bf45-7cf0c6a8bd6e"
+					(reference "C18")
+					(unit 1)
+				)
+			)
 		)
 	)
@@
 			)
 		)
-		(property "Value" "100k"
+		(property "Value" "1M"
 			(at 95.25 30.48 90)
 			(show_name no)
@@
 	)
 	(symbol
+		(lib_id "Device:C")
+		(at 63.5 48.26 90)
+		(unit 1)
+		(body_style 1)
+		(exclude_from_sim no)
+		(in_bom yes)
+		(on_board yes)
+		(in_pos_files yes)
+		(dnp no)
+		(fields_autoplaced yes)
+		(property "Reference" "C11"
+			(at 63.5 40.64 90)
+			(show_name no)
+			(do_not_autoplace no)
+			(effects
+				(font
+					(size 1.27 1.27)
+				)
+			)
+		)
+		(property "Value" "3.3u"
+			(at 63.5 43.18 90)
+			(show_name no)
+			(do_not_autoplace no)
+			(effects
+				(font
+					(size 1.27 1.27)
+				)
+			)
+		)
+		(property "Footprint" "Capacitor_SMD:C_1206_3216Metric"
+			(at 67.31 47.2948 0)
+			(hide yes)
+			(show_name no)
+			(do_not_autoplace no)
+			(effects
+				(font
+					(size 1.27 1.27)
+				)
+			)
+		)
+		(property "Datasheet" ""
+			(at 63.5 48.26 0)
+			(hide yes)
+			(show_name no)
+			(do_not_autoplace no)
+			(effects
+				(font
+					(size 1.27 1.27)
+				)
+			)
+		)
+		(property "Description" "Unpolarized capacitor"
+			(at 63.5 48.26 0)
+			(hide yes)
+			(show_name no)
+			(do_not_autoplace no)
+			(effects
+				(font
+					(size 1.27 1.27)
+				)
+			)
+		)
+		(pin "1"
+		)
+		(pin "2"
+		)
+		(instances
+			(project "LEOS-efm"
+				(path "/3703ddf2-8141-438d-86a8-1eaec9672d0d/63365fd5-9ed8-4ace-be7f-754e14efcbff"
+					(reference "C11")
+					(unit 1)
+				)
+				(path "/3703ddf2-8141-438d-86a8-1eaec9672d0d/fd5efc03-4429-4730-bf45-7cf0c6a8bd6e"
+					(reference "C16")
+					(unit 1)
+				)
+			)
+		)
+	)
+	(symbol
 		(lib_id "power:VDD")
 		(at 154.94 53.34 0)
@@
 			)
 		)
-		(property "Value" "1k"
+		(property "Value" "10k"
 			(at 73.66 44.45 90)
 			(show_name no)
@@
 			)
 		)
-		(property "Value" "1k"
+		(property "Value" "10k"
 			(at 73.66 77.47 90)
 			(show_name no)
@@
 			)
 		)
-		(property "Value" "100k"
+		(property "Value" "1M"
 			(at 95.25 64.77 90)
 			(show_name no)
